File: NRF905_SENDER/HW/NRF_SENDER.kicad_pcb (KiCad board)
At the start: 2 copper layers, 76 x 51 mm, 56 parts, among them J1 Conn_01x06_Male, J2 Conn_Coaxial, Q1 IRLML6402, SW1 SW_Push, SW2 SW_Push, U1 STM32L031F6Px, U2 BME280, U3 NRF905, Y1 Crystal

Commit message: Изменена структура проека. Добавлен шаблон проекта для ESP32. Изменение в схемотехнике WIFI модуль с ESP-07 изменени на ESP32 WROVER-IB
Parts:
- C19: value C -> 10 uf
Connections:
- U3 pad 33: GND -> (no net)
Changed lines of the file:
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@@
     (pad "" smd roundrect (at -1.2 0 180) (size 0.97 0.97) (layers F.Paste) (roundrect_rratio 0.25))
     (pad "" smd roundrect (at -1.2 -1.2 180) (size 0.97 0.97) (layers F.Paste) (roundrect_rratio 0.25))
-    (pad 33 smd roundrect (at 0 0 180) (size 3.6 3.6) (layers F.Cu F.Mask) (roundrect_rratio 0.06900000000000001)
-      (net 7 GND))
+    (pad 33 smd roundrect (at 0 0 180) (size 3.6 3.6) (layers F.Cu F.Mask) (roundrect_rratio 0.06900000000000001))
     (model ${KISYS3DMOD}/Package_DFN_QFN.3dshapes/QFN-32-1EP_5x5mm_P0.5mm_EP3.6x3.6mm.wrl
       (at (xyz 0 0 0))
@@
       (effects (font (size 1 1) (thickness 0.15)))
     )
-    (fp_text value C (at 0 1.43) (layer F.Fab)
+    (fp_text value "10 uf" (at 0 1.43) (layer F.Fab)
       (effects (font (size 1 1) (thickness 0.15)))
     )
@@
   (segment (start 85.598 59.682) (end 85.598 60.198) (width 0.2) (layer F.Cu) (net 6))
   (segment (start 85.89 59.39) (end 85.598 59.682) (width 0.2) (layer F.Cu) (net 6))
-  (segment (start 85.89 57.425) (end 85.89 59.39) (width 0.2) (layer F.Cu) (net 6))
+  (segment (start 85.89 57.425) (end 85.89 59.39) (width 0.2) (layer F.Cu) (net 6) (status 10))
   (segment (start 71.285 54.23) (end 71.28 54.225) (width 0.2) (layer F.Cu) (net 7))
   (segment (start 71.285 54.55) (end 71.285 54.23) (width 0.2) (layer F.Cu) (net 7))
@@
   (segment (start 73.44 54.555) (end 73.44 52.04) (width 0.2) (layer F.Cu) (net 7) (status 10))
   (segment (start 73.44 52.04) (end 73.34 51.94) (width 0.2) (layer F.Cu) (net 7))
+  (segment (start 77.57 59.68) (end 77.57 57.98) (width 0.2) (layer F.Cu) (net 7) (status 30))
+  (segment (start 77.07 58.48) (end 78.32 57.23) (width 0.2) (layer F.Cu) (net 7) (status 30))
+  (segment (start 77.07 59.68) (end 77.07 58.48) (width 0.2) (layer F.Cu) (net 7) (status 30))
+  (via (at 77.14 56.24) (size 0.6) (drill 0.3) (layers F.Cu B.Cu) (net 7) (status 30))
+  (via (at 78.14 56.24) (size 0.6) (drill 0.3) (layers F.Cu B.Cu) (net 7) (status 30))
+  (via (at 79.14 56.24) (size 0.6) (drill 0.3) (layers F.Cu B.Cu) (net 7) (status 30))
+  (via (at 79.14 57.24) (size 0.6) (drill 0.3) (layers F.Cu B.Cu) (net 7) (status 30))
+  (via (at 78.14 57.24) (size 0.6) (drill 0.3) (layers F.Cu B.Cu) (net 7) (status 30))
+  (via (at 77.14 57.24) (size 0.6) (drill 0.3) (layers F.Cu B.Cu) (net 7) (status 30))
+  (via (at 77.14 58.24) (size 0.6) (drill 0.3) (layers F.Cu B.Cu) (net 7) (status 30))
+  (via (at 78.14 58.24) (size 0.6) (drill 0.3) (layers F.Cu B.Cu) (net 7) (status 30))
   (via (at 79.14 58.24) (size 0.6) (drill 0.3) (layers F.Cu B.Cu) (net 7) (status 30))
-  (via (at 78.14 58.24) (size 0.6) (drill 0.3) (layers F.Cu B.Cu) (net 7) (status 30))
-  (via (at 77.14 58.24) (size 0.6) (drill 0.3) (layers F.Cu B.Cu) (net 7) (status 30))
-  (via (at 77.14 57.24) (size 0.6) (drill 0.3) (layers F.Cu B.Cu) (net 7) (status 30))
-  (via (at 78.14 57.24) (size 0.6) (drill 0.3) (layers F.Cu B.Cu) (net 7) (status 30))
-  (via (at 79.14 57.24) (size 0.6) (drill 0.3) (layers F.Cu B.Cu) (net 7) (status 30))
-  (via (at 79.14 56.24) (size 0.6) (drill 0.3) (layers F.Cu B.Cu) (net 7) (status 30))
-  (via (at 78.14 56.24) (size 0.6) (drill 0.3) (layers F.Cu B.Cu) (net 7) (status 30))
-  (via (at 77.14 56.24) (size 0.6) (drill 0.3) (layers F.Cu B.Cu) (net 7) (status 30))
-  (segment (start 77.07 59.68) (end 77.07 58.48) (width 0.2) (layer F.Cu) (net 7) (status 30))
-  (segment (start 77.07 58.48) (end 78.32 57.23) (width 0.2) (layer F.Cu) (net 7) (status 30))
-  (segment (start 77.57 59.68) (end 77.57 57.98) (width 0.2) (layer F.Cu) (net 7) (status 30))
+  (segment (start 80.07 55.48) (end 78.32 57.23) (width 0.2) (layer F.Cu) (net 7) (status 20))
+  (segment (start 76.57 55.48) (end 78.32 57.23) (width 0.2) (layer F.Cu) (net 7) (status 20))
+  (segment (start 76.57 58.98) (end 78.32 57.23) (width 0.2) (layer F.Cu) (net 7) (status 20))
+  (segment (start 79.07 57.98) (end 78.32 57.23) (width 0.2) (layer F.Cu) (net 7) (status 30))
+  (segment (start 79.07 59.68) (end 79.07 57.98) (width 0.2) (layer F.Cu) (net 7) (status 30))
+  (segment (start 78.57 57.48) (end 78.32 57.23) (width 0.2) (layer F.Cu) (net 7) (status 30))
+  (segment (start 78.57 59.68) (end 78.57 57.48) (width 0.2) (layer F.Cu) (net 7) (status 30))
+  (segment (start 78.07 57.48) (end 78.32 57.23) (width 0.2) (layer F.Cu) (net 7) (status 30))
+  (segment (start 78.07 59.68) (end 78.07 57.48) (width 0.2) (layer F.Cu) (net 7) (status 30))
   (segment (start 77.57 57.98) (end 78.32 57.23) (width 0.2) (layer F.Cu) (net 7) (status 30))
-  (segment (start 78.07 59.68) (end 78.07 57.48) (width 0.2) (layer F.Cu) (net 7) (status 30))
-  (segment (start 78.07 57.48) (end 78.32 57.23) (width 0.2) (layer F.Cu) (net 7) (status 30))
-  (segment (start 78.57 59.68) (end 78.57 57.48) (width 0.2) (layer F.Cu) (net 7) (status 30))
-  (segment (start 78.57 57.48) (end 78.32 57.23) (width 0.2) (layer F.Cu) (net 7) (status 30))
-  (segment (start 79.07 59.68) (end 79.07 57.98) (width 0.2) (layer F.Cu) (net 7) (status 30))
-  (segment (start 79.07 57.98) (end 78.32 57.23) (width 0.2) (layer F.Cu) (net 7) (status 30))
-  (segment (start 76.57 58.98) (end 78.32 57.23) (width 0.2) (layer F.Cu) (net 7) (status 20))
-  (segment (start 76.57 55.48) (end 78.32 57.23) (width 0.2) (layer F.Cu) (net 7) (status 20))
-  (segment (start 80.07 55.48) (end 78.32 57.23) (width 0.2) (layer F.Cu) (net 7) (status 20))
   (segment (start 92.71 61.214) (end 92.71 62.738) (width 0.5) (layer F.Cu) (net 8) (status 30))
   (segment (start 92.71 62.738) (end 92.71 64.262) (width 0.5) (layer F.Cu) (net 8) (status 30))
@@
   (segment (start 79.57 53.79) (end 80.47999 52.88001) (width 0.2) (layer F.Cu) (net 25))
   (segment (start 79.57 54.78) (end 79.57 53.79) (width 0.2) (layer F.Cu) (net 25) (status 10))
-  (segment (start 85.84 53.582) (end 85.84 56.405) (width 0.2) (layer F.Cu) (net 25))
-  (segment (start 85.84 56.405) (end 85.89 56.455) (width 0.2) (layer F.Cu) (net 25))
+  (segment (start 85.84 53.582) (end 85.84 56.405) (width 0.2) (layer F.Cu) (net 25) (status 20))
+  (segment (start 85.84 56.405) (end 85.89 56.455) (width 0.2) (layer F.Cu) (net 25) (status 30))
   (segment (start 85.478 53.22) (end 85.84 53.582) (width 0.2) (layer F.Cu) (net 25))
   (segment (start 83.92 53.22) (end 85.478 53.22) (width 0.2) (layer F.Cu) (net 25))

Commit message: Добавлена тестовая прошивка для Sender. Исправленны ошибки в печатной плате
Parts:
- J1: footprint Connector_PinSocket_1.27mm:PinSocket_1x06_P1.27mm_Vertical -> Connector_PinSocket_2.54mm:PinSocket_1x06_P2.54mm_Vertical
- SW1, SW2: footprint push_button:push -> Button_Switch_SMD:SW_SPST_EVQP2
- moved SW2 11.0 mm to (87.5, 88.9), turned to 180 degrees
- moved SW1 10.1 mm to (76.4, 88.9)
- moved C19 6.93 mm to (113.9, 57.3)
- moved C15 5.30 mm to (111.0, 65.6), turned to 270 degrees
- moved D2 1.36 mm to (111.2, 61.9), turned to 90 degrees
- moved J1 0.77 mm to (71.5, 73.0)
Connections:
- U3 pad 33: (no net) -> GND
Routing:
- net GND: track 184.7 -> 158.3 mm
- net Net-(C3-Pad1): track 25.5 -> 35.8 mm
- net Net-(D2-Pad5): track 19.7 -> 10.5 mm, vias 3 -> 0
- net /SP_EN: track 48.5 -> 57.4 mm, vias 2 -> 4
- net /PWR_L: track 57.0 -> 48.6 mm
- net Net-(J1-Pad3): track 16.5 -> 19.3 mm
- net /KEY: track 16.3 -> 16.9 mm
- net Net-(J1-Pad2): track 11.3 -> 11.8 mm
Other:
- outline, holes or cut-outs redrawn
