File: NRF905_SENDER/HW/NRF_SENDER.sch (KiCad schematic (older format))
At the start: 23 parts, among them J1 Conn_01x06_Male, SW1 SW_Push, SW2 SW_Push, U1 STM32L031F6Px

Commit message: Добавлена тестовая прошивка для Sender. Исправленны ошибки в печатной плате
Parts:
- J1: footprint Connector_PinSocket_1.27mm:PinSocket_1x06_P1.27mm_Vertical -> Connector_PinSocket_2.54mm:PinSocket_1x06_P2.54mm_Vertical
- SW1, SW2: footprint push_button:push -> Button_Switch_SMD:SW_SPST_EVQP2
Changed lines of the file:
@@
 F 0 "SW2" H 7150 5085 50  0000 C CNN
 F 1 "SW_Push" H 7150 4994 50  0000 C CNN
-F 2 "push_button:push" H 7150 5000 50  0001 C CNN
+F 2 "Button_Switch_SMD:SW_SPST_EVQP2" H 7150 5000 50  0001 C CNN
 F 3 "~" H 7150 5000 50  0001 C CNN
 	1    7150 4800
@@
 F 0 "SW1" V 3246 2202 50  0000 R CNN
 F 1 "SW_Push" V 3155 2202 50  0000 R CNN
-F 2 "push_button:push" H 3200 2450 50  0001 C CNN
+F 2 "Button_Switch_SMD:SW_SPST_EVQP2" H 3200 2450 50  0001 C CNN
 F 3 "~" H 3200 2450 50  0001 C CNN
 	1    3200 2250
@@
 F 0 "J1" H 3972 5882 50  0000 R CNN
 F 1 "Conn_01x06_Male" H 3972 5973 50  0000 R CNN
-F 2 "Connector_PinSocket_1.27mm:PinSocket_1x06_P1.27mm_Vertical" H 4000 6000 50  0001 C CNN
+F 2 "Connector_PinSocket_2.54mm:PinSocket_1x06_P2.54mm_Vertical" H 4000 6000 50  0001 C CNN
 F 3 "~" H 4000 6000 50  0001 C CNN
 	1    4000 6000
