File: NRF905_RECIVER/HW/ESP-Wrover IB.sch (KiCad schematic (older format))
At the start: 13 parts, among them J2 USB_B_Micro, U3 CP2102N-A01-GQFN28

Commit message: new scematics. New PCB.
Parts:
- A1: symbol ESP32-WROVER-I:ESP32-WROVER-I -> RECIVER_NRF-rescue:ESP32-WROVER-I-ESP32-WROVER-I
Changed lines of the file:
@@
 Connection ~ 6200 1850
 $Comp
-L ESP32-WROVER-I:ESP32-WROVER-I A1
+L RECIVER_NRF-rescue:ESP32-WROVER-I-ESP32-WROVER-I A1
 U 1 1 5F81E405
 P 4350 3150
+AR Path="/5F81E405" Ref="A1"  Part="1"
+AR Path="/5F662950/5F81E405" Ref="A1"  Part="1"
 F 0 "A1" H 3950 4550 50  0000 C CNN
 F 1 "ESP32-WROVER-I" H 3850 4450 50  0000 C CNN
