File: NRF905_SENDER/HW_433/power.sch (KiCad schematic (older format))
At the start: 11 parts, among them Q1 IRLML6402

Commit message: new scematics. New PCB.
Parts:
- renumbered R17 to R18, R18 to R19, R19 to R20, D2 to U4
Changed lines of the file:
@@
 $EndDescr
 $Comp
-L max1724:MAX1724 D2
+L max1724:MAX1724 U4
 U 1 1 5EB552F6
 P 5450 3250
-F 0 "D2" H 5700 3425 50  0000 C CNN
+F 0 "U4" H 5700 3425 50  0000 C CNN
 F 1 "MAX1724" H 5700 3334 50  0000 C CNN
 F 2 "modules:TSOT" H 5450 3250 50  0001 C CNN
@@
 Connection ~ 5300 2800
 $Comp
-L Device:R R17
+L Device:R R18
 U 1 1 5EB581FA
 P 5200 4100
-F 0 "R17" V 4993 4100 50  0000 C CNN
+F 0 "R18" V 4993 4100 50  0000 C CNN
 F 1 "10 k" V 5084 4100 50  0000 C CNN
 F 2 "Resistor_SMD:R_0603_1608Metric_Pad1.05x0.95mm_HandSolder" V 5130 4100 50  0001 C CNN
@@
 Connection ~ 7000 2800
 $Comp
-L Device:R R19
+L Device:R R20
 U 1 1 5EB5A9B2
 P 7800 3550
-F 0 "R19" H 7870 3596 50  0000 L CNN
+F 0 "R20" H 7870 3596 50  0000 L CNN
 F 1 "10 k" H 7870 3505 50  0000 L CNN
 F 2 "Resistor_SMD:R_0603_1608Metric_Pad1.05x0.95mm_HandSolder" V 7730 3550 50  0001 C CNN
@@
 $EndComp
 $Comp
-L Device:R R18
+L Device:R R19
 U 1 1 5EB5B023
 P 7350 3100
-F 0 "R18" H 7420 3146 50  0000 L CNN
+F 0 "R19" H 7420 3146 50  0000 L CNN
 F 1 "100 k" H 7420 3055 50  0000 L CNN
 F 2 "Resistor_SMD:R_0603_1608Metric_Pad1.05x0.95mm_HandSolder" V 7280 3100 50  0001 C CNN
