File: NRF905_SENDER/HW_433/NRF905.sch (KiCad schematic (older format))
At the start: 19 parts, among them J2 Conn_Coaxial, U3 NRF905, Y1 Crystal

Commit message: new scematics. New PCB.
Parts:
- renumbered R20 to R17
Changed lines of the file:
@@
 Connection ~ 2150 4200
 $Comp
-L Device:R R20
+L Device:R R17
 U 1 1 5EB9E4FF
 P 2750 4350
-F 0 "R20" H 2820 4396 50  0000 L CNN
+F 0 "R17" H 2820 4396 50  0000 L CNN
 F 1 "1 M" H 2820 4305 50  0000 L CNN
 F 2 "Resistor_SMD:R_0402_1005Metric" V 2680 4350 50  0001 C CNN

Commit message: Change ESP32
Parts:
- U3: symbol _wireless:NRF905 -> NRF_SENDER-rescue:NRF905-_wireless
Changed lines of the file:
@@
 	2600 2700 3050 2700
 $Comp
-L _wireless:NRF905 U3
+L NRF_SENDER-rescue:NRF905-_wireless U3
 U 1 1 5EBD3534
 P 4300 3200
