File: NRF905_SENDER/HW_433/NRF_SENDER.kicad_pcb (KiCad board)
At the start: 2 copper layers, 76 x 51 mm, 54 parts, among them J1 SWD, J2 Conn_Coaxial, Q1 IRLML6402, SW1 SW_Push, SW2 SW_Push, U1 STM32L031F6Px, U2 BME280, U3 NRF905, Y1 Crystal

Commit message: new scematics. New PCB.
Parts:
- removed the R3 at (92.1, 64.3)
- removed the R4 at (92.1, 66.0)
- removed the R5 at (87.0, 57.0)
- removed the R7 at (92.1, 60.9)
- added C20: 0.1 uf, Capacitor_SMD:C_0603_1608Metric_Pad1.05x0.95mm_HandSolder, F.Cu at (88.5, 76.7)
- added C21: 0.1 uf, Capacitor_SMD:C_0603_1608Metric_Pad1.05x0.95mm_HandSolder, F.Cu at (92.0, 69.8)
- added C22: 0.1 uf, Capacitor_SMD:C_0603_1608Metric_Pad1.05x0.95mm_HandSolder, F.Cu at (82.1, 63.0)
- added C23: 0.1 uf, Capacitor_SMD:C_0603_1608Metric_Pad1.05x0.95mm_HandSolder, F.Cu at (80.1, 74.5)
- added D1: LED, LED_SMD:LED_0603_1608Metric_Pad1.05x0.95mm_HandSolder, F.Cu at (73.1, 66.7)
- added D2: LED, LED_SMD:LED_0603_1608Metric_Pad1.05x0.95mm_HandSolder, F.Cu at (73.2, 68.6)
- added R10: 120, Resistor_SMD:R_0603_1608Metric_Pad1.05x0.95mm_HandSolder, F.Cu at (77.2, 70.6)
- added R11: 120, Resistor_SMD:R_0603_1608Metric_Pad1.05x0.95mm_HandSolder, F.Cu at (77.2, 72.4)
- added R12: 120, Resistor_SMD:R_0603_1608Metric_Pad1.05x0.95mm_HandSolder, F.Cu at (83.6, 78.0)
- added R14: 330, Resistor_SMD:R_0603_1608Metric_Pad1.05x0.95mm_HandSolder, F.Cu at (77.2, 66.7)
- added R15: 330, Resistor_SMD:R_0603_1608Metric_Pad1.05x0.95mm_HandSolder, F.Cu at (77.2, 68.6)
- R2, R8, R9: value 10 k -> 120
- U1: value STM32L031F6Px -> STM32L051C6Tx; footprint Package_SO:TSSOP-20_4.4x6.5mm_P0.65mm -> Package_QFP:LQFP-48_7x7mm_P0.5mm
- moved R2 26.8 mm to (86.7, 56.3), turned to 90 degrees
- moved R9 11.9 mm to (88.5, 56.3), turned to 270 degrees
- moved C2 9.60 mm to (76.3, 77.6), turned to 180 degrees
- moved R6 8.32 mm to (85.8, 62.6)
- moved U1 7.79 mm to (85.8, 70.3), turned to 180 degrees
- moved R4 6.79 mm to (89.3, 62.6)
- moved R8 6.52 mm to (90.4, 56.3), turned to 270 degrees
- moved R5 6.29 mm to (87.5, 62.6)
- moved R3 6.14 mm to (91.0, 62.6)
- moved R7 1.75 mm to (84.0, 62.6)
- moved SW1 0.62 mm to (77.1, 88.9)
- renumbered R15 to R13, R20 to R17, R17 to R18, R18 to R19, R19 to R20, R10 to R3, R11 to R4, R12 to R5, R13 to R6, R14 to R7, D2 to U4
Connections:
- C1 pad 1: /POWER/POWER_MCU -> /VDD
- C16 pad 1: /POWER/POWER_MCU -> /VDD
- C19 pad 1: /POWER/POWER_MCU -> /VDD
- C2 pad 1: /POWER/POWER_MCU -> /VDD
- D3 pad 1: /POWER/POWER_MCU -> /VDD
- J1 pad 1: /POWER/POWER_MCU -> /VDD
- Q1 pad 2: /POWER/POWER_MCU -> /VDD
- R1 pad 1: /POWER/POWER_MCU -> /VDD
- R13 pad 1: /POWER/POWER_MCU -> /VDD
- R19 pad 1: /POWER/POWER_MCU -> /VDD
- R2 pad 2: GND -> /DR
- R3 pad 1: /CSK -> /CE
- R4 pad 1: /MISO -> /TX_EN
- R4 pad 2: Net-(R11-Pad2) -> Net-(R4-Pad2)
- R5 pad 1: /MOSI -> /CS_BME
- R5 pad 2: Net-(R12-Pad2) -> Net-(R5-Pad2)
- R6 pad 1: /CS_BME -> /CS_NRF
- R6 pad 2: Net-(R13-Pad2) -> Net-(R6-Pad2)
- R7 pad 1: /CE -> /CSK
- R7 pad 2: Net-(R14-Pad2) -> Net-(R7-Pad2)
- R8 pad 1: /POWER/POWER_MCU -> /MISO
- R8 pad 2: Net-(R12-Pad2) -> Net-(R8-Pad2)
- R9 pad 1: /POWER/POWER_MCU -> /MOSI
- R9 pad 2: Net-(R11-Pad2) -> Net-(R9-Pad2)
- U1 pad 1: Net-(R2-Pad1) -> (no net)
- U1 pad 10: /DR -> /PWR_L
- U1 pad 12: Net-(R11-Pad2) -> Net-(R4-Pad2)
- U1 pad 13: Net-(R12-Pad2) -> Net-(R5-Pad2)
- U1 pad 14: Net-(R4-Pad1) -> Net-(R6-Pad2)
- U1 pad 15: GND -> Net-(R7-Pad2)
- U1 pad 16: /POWER/POWER_MCU -> Net-(R8-Pad2)
- U1 pad 17: Net-(R13-Pad2) -> Net-(R9-Pad2)
- U1 pad 18: Net-(R14-Pad2) -> Net-(R2-Pad1)
- U1 pad 19: Net-(J1-Pad4) -> (no net)
- U1 pad 2: /PWR -> (no net)
- U1 pad 20: Net-(J1-Pad2) -> (no net)
- U1 pad 3: /TX_EN -> (no net)
- U1 pad 4: Net-(C3-Pad1) -> (no net)
- U1 pad 5: /POWER/POWER_MCU -> (no net)
- U1 pad 6: /PWR_L -> (no net)
- U1 pad 7: /SP_EN -> GND
- U1 pad 8: /KEY -> GND
- U1 pad 9: /MP_EN -> /VDD
- U4 pad 4: /POWER/POWER_MCU -> /VDD
Routing:
- net /VDD: track 0.00 -> 146.9 mm, vias 0 -> 5
- net /POWER/POWER_MCU: track 121.3 -> 0.00 mm, vias 7 -> 0
- net /DR: track 42.1 -> 5.97 mm, vias 2 -> 0
- net /TX_EN: track 39.5 -> 11.3 mm, vias 2 -> 0
- net Net-(R13-Pad2): track 27.1 -> 0.00 mm, vias 2 -> 0
- net Net-(R11-Pad2): track 28.9 -> 4.29 mm, vias 1 -> 0
- net Net-(R12-Pad2): track 27.0 -> 2.61 mm, vias 2 -> 0
- net Net-(R4-Pad1): track 22.8 -> 0.00 mm, vias 2 -> 0
- net /KEY: track 18.1 -> 39.6 mm, vias 0 -> 2
- net Net-(R3-Pad2): track 23.5 -> 6.02 mm, vias 2 -> 0
- net Net-(R9-Pad2): track 0.00 -> 16.5 mm, vias 0 -> 2
- net Net-(R8-Pad2): track 0.00 -> 15.8 mm, vias 0 -> 2
- net GND: track 156.7 -> 142.7 mm, vias 106 -> 104
- net /MP_EN: track 4.48 -> 17.7 mm, vias 0 -> 2
- net Net-(J1-Pad4): track 12.8 -> 25.0 mm
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
Commit message: Change ESP32
Routing:
- net GND: track 142.7 -> 157.1 mm
